File: Hardware/main_board/main_board.kicad_pcb (KiCad board)
At the start: 6 copper layers, 95.4 x 36.1 mm, 234 parts, among them J1 BATT, J2 LCD, J3 BACK_LIGHT, J4 SD, J5 NFC, J6 EXT1, J7 EXT0, J8 USB_C, Q1 DMN313DLT, SW1 OK, SW2 BACK, SW3 RIGHT, SW4 LEFT, SW5 UP, SW6 DOWN, T1 B0310J50100AHF, U1 STM32WB55RGVx, U10 BGS13S4N9E6327XTSA1, U11 NC7SZ32M5X, U12 LP5562TMX, U2 BQ27220YZFR, U3 BQ25896RTWR, U4 RS3221-3.3YF3, U5 LM66100DCK, U6 LM3281YFQR, U7 LM3281YFQR, U8 CC1101RGP, U9 BGS13S4N9E6327XTSA1, Y1 32MHz, Y2 32.768K, Y3 26MHz

Commit message: layout: finish the layout initially
Parts:
- removed FB1, FB2: 120R@100MHz, Inductor_SMD:L_0603_1608Metric
- moved C81 22.4 mm to (124.5, 100.1)
- moved R29 1.02 mm to (182.1, 113.9), turned to 90 degrees
Connections:
- C29 pad 1: GNDP -> GND
- C30 pad 1: GNDP -> GND
- C31 pad 1: GNDP -> GND
- C34 pad 1: GNDP -> GND
- C35 pad 1: GNDP -> GND
- C36 pad 1: GNDP -> GND
- C37 pad 1: GNDP -> GND
- C38 pad 1: GNDP -> GND
- C39 pad 1: GNDP -> GND
- U6 pad C2: GNDP -> GND
- U7 pad C2: GNDP -> GND
Routing:
- net /CC1101/SPI_R_SCK: track 1.89 -> 59.9 mm, vias 2 -> 4
- net /MCU/iBTN: track 3.02 -> 54.1 mm, vias 1 -> 5
- net BAT: track 32.6 -> 83.6 mm, vias 3 -> 4
- net /CC1101/SPI_R_MISO: track 1.61 -> 49.7 mm, vias 1 -> 3
- net /CC1101/SPI_R_MOSI: track 0.75 -> 48.0 mm, vias 1 -> 5
- net /Buttons/BUTTON_BACK: track 0.00 -> 43.9 mm, vias 0 -> 3
- net /CC1101/CC1101_CS: track 1.14 -> 42.2 mm, vias 1 -> 2
- net /MCU/PC1: track 2.00 -> 42.3 mm
- net /MCU/NFC_CS: track 0.70 -> 35.7 mm, vias 1 -> 3
- net /MCU/PC0: track 2.31 -> 36.7 mm
- net /Buttons/BUTTON_RIGHT: track 0.00 -> 33.6 mm, vias 0 -> 1
- net /Buttons/BUTTON_OK: track 0.74 -> 34.3 mm, vias 1 -> 2
- net /MCU/SPI_D_MISO: track 3.59 -> 36.9 mm, vias 2 -> 3
- net /MCU/SD_CD: track 1.81 -> 34.8 mm, vias 0 -> 2
- net Net-(D8-A): track 0.00 -> 32.4 mm, vias 0 -> 3
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- removed copper zone on In2.Cu, net GND
- removed copper zone on B.Cu, net GNDP
- removed copper zone on In1.Cu, net GNDP
- removed copper zone on In2.Cu, net GNDP
- removed copper zone on In3.Cu, net GNDP
