File: Hardware/main_board/periphery.kicad_sch (KiCad schematic)
At the start: 66 parts, among them J4 SD, J5 NFC, J6 EXT1, J7 EXT0, U12 LP5562TMX

Commit message: sch: change sd card footprint
Parts:
- J4: footprint Library:TF-101A-P3 -> Library:TF-SMD_TF-110
Changed lines of the file:
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@@
 			)
 		)
-		(property "Footprint" "Library:TF-101A-P3"
+		(property "Footprint" "Library:TF-SMD_TF-110"
 			(at 292.1 34.29 0)
 			(effects
