File: Hardware/nfc_rfid/nfc_rfid.kicad_pcb (KiCad board)
At the start: 4 copper layers, 74.1 x 32 mm, 158 parts, among them IC1 ST25R3916-AQWT, IC2 FAN48610UC50X, J1 BW0033AG-L3.4W0.9H1.8, J2 BW0033AG-L3.4W0.9H1.8, J3 HC-FPC-05-09-18RLTAG, J4 +, J5 -, J6 AFH34-S06FIA-1H, J7 BW0033AG-L3.4W0.9H1.8, J8 BW0033AG-L3.4W0.9H1.8, Q1 AO3400A, Q2 DMN2004TK-7, Q3 DMP2004TK-7, Q4 DMN2004TK-7, Q5 DMN5L06TK-7, U1 LMV358AIDGKR, U2 LMV331IDCKR, U3 LMV358AIDGKR, Y1 CF4027M12010001

Commit message: PCB: nfc_rfid: adjust vibro touch point
Parts:
- moved J4 0.61 mm to (139.8, 69.2)
- moved J5 0.61 mm to (142.3, 69.2)
Routing:
- net Net-(D1-A): track 18.7 -> 19.7 mm
Changed lines of the file:
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@@
 	(footprint "Library:TestPoint_Pad_3.0x2.0mm_round_corner_no_silkscreen"
 		(layer "F.Cu")
-		(at 139.7508 69.7992 90)
+		(at 139.7762 69.1896 90)
 		(descr "SMD rectangular pad as test Point, square 3.0mm side length")
 		(tags "test point SMD pad rectangle square")
@@
 		(attr exclude_from_pos_files exclude_from_bom)
 		(fp_rect
-			(start -1.55 -1.05)
-			(end 1.55 1.05)
+			(start -2.55 -1.05)
+			(end 2.575 1.05)
 			(stroke
 				(width 0.05)
@@
 		(pad "1" smd roundrect
 			(at 0 0 90)
-			(size 3 2)
+			(size 5 2)
 			(layers "F.Cu" "F.Mask")
 			(roundrect_rratio 0.4)
@@
 	(footprint "Library:TestPoint_Pad_3.0x2.0mm_round_corner_no_silkscreen"
 		(layer "F.Cu")
-		(at 142.24 69.7992 90)
+		(at 142.2654 69.1896 90)
 		(descr "SMD rectangular pad as test Point, square 3.0mm side length")
 		(tags "test point SMD pad rectangle square")
@@
 		(attr exclude_from_pos_files exclude_from_bom)
 		(fp_rect
-			(start -1.55 -1.05)
-			(end 1.55 1.05)
+			(start -2.6 -1.05)
+			(end 2.6 1.05)
 			(stroke
 				(width 0.05)
@@
 		(pad "1" smd roundrect
 			(at 0 0 90)
-			(size 3 2)
+			(size 5 2)
 			(layers "F.Cu" "F.Mask")
 			(roundrect_rratio 0.4)
@@
 	)
 	(segment
-		(start 137.7188 61.6644)
-		(end 135.8446 59.7902)
+		(start 138.9126 65.4558)
+		(end 141.0316 65.4558)
 		(width 0.5588)
 		(layer "F.Cu")
@@
 	(segment
 		(start 137.7188 64.262)
-		(end 142.24 68.7832)
+		(end 138.9126 65.4558)
 		(width 0.5588)
 		(layer "F.Cu")
@@
 	)
 	(segment
-		(start 135.8446 57.0992)
-		(end 135.8446 55.8492)
+		(start 137.7188 61.6644)
+		(end 135.8446 59.7902)
 		(width 0.5588)
 		(layer "F.Cu")
@@
 	)
 	(segment
-		(start 142.24 68.7832)
-		(end 142.24 69.7992)
-		(width 0.254)
+		(start 141.0316 65.4558)
+		(end 142.2654 66.6896)
+		(width 0.5588)
+		(layer "F.Cu")
+		(net 37)
+	)
+	(segment
+		(start 135.8446 57.0992)
+		(end 135.8446 55.8492)
+		(width 0.5588)
 		(layer "F.Cu")
 		(net 37)
@@
 		(net 37)
 	)
+	(segment
+		(start 137.7188 64.262)
+		(end 137.7188 63.9572)
+		(width 0.5588)
+		(layer "F.Cu")
+		(net 37)
+	)
+	(segment
+		(start 142.2654 66.6896)
+		(end 142.2654 69.1896)
+		(width 0.5588)
+		(layer "F.Cu")
+		(net 37)
+	)
 	(via
 		(at 136.398 55.2958)
@@
 	)
 	(zone
-		(net 10)
-		(net_name "Net-(C11-Pad1)")
+		(net 11)
+		(net_name "/NFC/RFI_N")
 		(layer "F.Cu")
 		(name "$teardrop_padvia$")
 		(hatch full 0.1)
-		(priority 30001)
+		(priority 30004)
 		(attr
 			(teardrop
@@
 		(polygon
 			(pts
-				(xy 124.4053 63.7626) (xy 124.4053 63.2038) (xy 123.844884 63.01535) (xy 123.3668 63.4281) (xy 123.74905 63.8656)
+				(xy 127.104 65.0298) (xy 127.404 65.0298) (xy 127.606118 64.716329) (xy 127.3784 64.4388) (xy 127.0984 64.6098)
 			)
 		)
 	)
 	(zone
-		(net 9)
-		(net_name "Net-(C12-Pad1)")
+		(net 52)
+		(net_name "Net-(IC1-RFO2)")
 		(layer "F.Cu")
 		(name "$teardrop_padvia$")
 		(hatch full 0.1)
-		(priority 30000)
+		(priority 30003)
 		(attr
 			(teardrop
@@
 		(polygon
 			(pts
-				(xy 124.4053 69.3674) (xy 124.4053 68.8086) (xy 123.74905 68.697) (xy 123.3668 69.1345) (xy 123.838817 69.551303)
+				(xy 122.3303 65.4558) (xy 122.3303 65.7606) (xy 122.902838 65.973949) (xy 123.3688 65.5531) (xy 122.890715 65.14035)
 			)
 		)
@@
 	)
 	(zone
-		(net 7)
-		(net_name "/NFC/RFI_P")
+		(net 49)
+		(net_name "Net-(IC1-RFO1)")
 		(layer "F.Cu")
 		(name "$teardrop_padvia$")
 		(hatch full 0.1)
-		(priority 30005)
+		(priority 30002)
 		(attr
 			(teardrop
@@
 		(polygon
 			(pts
-				(xy 127.404 67.5328) (xy 127.104 67.5328) (xy 127.0984 67.9528) (xy 127.3784 68.1238) (xy 127.606118 67.84627)
+				(xy 122.3303 66.8106) (xy 122.3303 67.1154) (xy 122.896782 67.426303) (xy 123.3688 67.0095) (xy 122.902838 66.588651)
 			)
 		)
 	)
 	(zone
-		(net 52)
-		(net_name "Net-(IC1-RFO2)")
+		(net 1)
+		(net_name "GND")
+		(layer "F.Cu")
+		(hatch edge 0.5)
+		(priority 1)
+		(connect_pads yes
+			(clearance 0.1016)
+		)
+		(min_thickness 0.2032)
+		(filled_areas_thickness no)
+		(fill yes
+			(thermal_gap 0.5)
+			(thermal_bridge_width 0.5)
+		)
+		(polygon
+			(pts
+				(xy 68.3768 45.5676) (xy 68.326 80.1116) (xy 147.32 80.0862) (xy 147.32 45.4406) (xy 147.32 45.466)
+			)
+		)
+	)
+	(zone
+		(net 7)
+		(net_name "/NFC/RFI_P")
 		(layer "F.Cu")
 		(name "$teardrop_padvia$")
 		(hatch full 0.1)
-		(priority 30003)
+		(priority 30005)
 		(attr
 			(teardrop
@@
 		(polygon
 			(pts
-				(xy 122.3303 65.4558) (xy 122.3303 65.7606) (xy 122.902838 65.973949) (xy 123.3688 65.5531) (xy 122.890715 65.14035)
+				(xy 127.404 67.5328) (xy 127.104 67.5328) (xy 127.0984 67.9528) (xy 127.3784 68.1238) (xy 127.606118 67.84627)
 			)
 		)
 	)
 	(zone
-		(net 1)
-		(net_name "GND")
+		(net 16)
+		(net_name "+5V")
 		(layer "F.Cu")
 		(hatch edge 0.5)
-		(priority 1)
+		(priority 4)
 		(connect_pads yes
 			(clearance 0.1016)
 		)
-		(min_thickness 0.2032)
+		(min_thickness 0.1524)
 		(filled_areas_thickness no)
 		(fill yes
@@
 		(polygon
 			(pts
-				(xy 68.3768 45.5676) (xy 68.326 80.1116) (xy 147.32 80.0862) (xy 147.32 45.4406) (xy 147.32 45.466)
+				(xy 109.2708 55.626) (xy 109.2708 58.2168) (xy 107.569 58.2168) (xy 107.569 56.6928) (xy 106.0196 56.6928)
+				(xy 106.0196 55.3974) (xy 106.9594 55.3974) (xy 107.2134 55.626)
 			)
 		)
 	)
 	(zone
-		(net 11)
-		(net_name "/NFC/RFI_N")
+		(net 9)
+		(net_name "Net-(C12-Pad1)")
 		(layer "F.Cu")
 		(name "$teardrop_padvia$")
 		(hatch full 0.1)
-		(priority 30004)
+		(priority 30000)
 		(attr
 			(teardrop
@@
 		(polygon
 			(pts
-				(xy 127.104 65.0298) (xy 127.404 65.0298) (xy 127.606118 64.716329) (xy 127.3784 64.4388) (xy 127.0984 64.6098)
+				(xy 124.4053 69.3674) (xy 124.4053 68.8086) (xy 123.74905 68.697) (xy 123.3668 69.1345) (xy 123.838817 69.551303)
 			)
 		)
 	)
 	(zone
-		(net 49)
-		(net_name "Net-(IC1-RFO1)")
+		(net 10)
+		(net_name "Net-(C11-Pad1)")
 		(layer "F.Cu")
 		(name "$teardrop_padvia$")
 		(hatch full 0.1)
-		(priority 30002)
+		(priority 30001)
 		(attr
 			(teardrop
@@
 		(polygon
 			(pts
-				(xy 122.3303 66.8106) (xy 122.3303 67.1154) (xy 122.896782 67.426303) (xy 123.3688 67.0095) (xy 122.902838 66.588651)
-			)
-		)
-	)
-	(zone
-		(net 16)
-		(net_name "+5V")
-		(layer "F.Cu")
-		(hatch edge 0.5)
-		(priority 4)
-		(connect_pads yes
-			(clearance 0.1016)
-		)
-		(min_thickness 0.1524)
-		(filled_areas_thickness no)
-		(fill yes
-			(thermal_gap 0.5)
-			(thermal_bridge_width 0.5)
-		)
-		(polygon
-			(pts
-				(xy 109.2708 55.626) (xy 109.2708 58.2168) (xy 107.569 58.2168) (xy 107.569 56.6928) (xy 106.0196 56.6928)
-				(xy 106.0196 55.3974) (xy 106.9594 55.3974) (xy 107.2134 55.626)
+				(xy 124.4053 63.7626) (xy 124.4053 63.2038) (xy 123.844884 63.01535) (xy 123.3668 63.4281) (xy 123.74905 63.8656)
 			)
 		)
